Commit message: origin done

File: urdf/robots/haique_description/urdf/haique.xacro (robot description, xacro)
@@ -133,5 +133,5 @@
     <xacro:macro name="thruster_macro1"
    	           params="thruster_id
-                        *joint_origin
+                        *origin
                         *axis
                         parent_link">
@@ -143,5 +143,5 @@
             dyn_time_constant="0.05"
             rotor_constant="0.00031">  <!-- This is a guess for now (same as Smilidon) -->
-        <xacro:insert_block name="joint_origin"/>
+        <xacro:insert_block name="origin"/>
         <xacro:insert_block name="axis"/>
         </xacro:thruster_module_first_order_basic_fcn_macro>
@@ -149,5 +149,5 @@
     <xacro:macro name="thruster_macro2"
    	           params="thruster_id
-                        *joint_origin
+                        *origin
                         *axis
                         parent_link">
@@ -159,5 +159,5 @@
             dyn_time_constant="0.05"
             rotor_constant="0.00031">  <!-- This is a guess for now (same as Smilidon) -->
-        <xacro:insert_block name="joint_origin"/>
+        <xacro:insert_block name="origin"/>
         <xacro:insert_block name="axis"/>
         </xacro:thruster_module_first_order_basic_fcn_macro>
@@ -165,6 +165,6 @@
     <!-- qianshang -->
     <xacro:thruster_macro1 thruster_id="0" parent_link="haique_link">
-        <joint_origin
-            xyz="-0.00013907 0.3405 0.04191"
+        <origin
+            xyz="-0.00013907 0.3405 0.04691"
             rpy="3.1383 0 1.5616" />
         <axis
@@ -173,7 +173,7 @@
     <!-- zuoshang -->
     <xacro:thruster_macro2 thruster_id="1" parent_link="zuo_link">
-        <joint_origin
-            xyz="0 -0.04109 0.2285"
-            rpy="1.5708 -1.3538 3.1416" />
+        <origin
+            xyz="0.006 -0.2285 -0.037 "
+            rpy="0 -0.21 0" />
         <axis
             xyz="0 0 -1" />
@@ -181,6 +181,6 @@
     <!-- houshang -->
     <xacro:thruster_macro1 thruster_id="2" parent_link="haique_link">
-        <joint_origin
-            xyz="0 -0.3005 0.04191"
+        <origin
+            xyz="0 -0.3005 0.04691"
             rpy="3.1416 0 1.5735" />
         <axis
@@ -189,7 +189,7 @@
     <!-- youshang -->
     <xacro:thruster_macro2 thruster_id="3" parent_link="you_link">
-        <joint_origin
-            xyz="-0.2285 0.03787 0"
-            rpy="-1.5708 0.1979 3.1416" />
+        <origin
+            xyz="0.02087 -0.2285 -0.03"
+            rpy="0 -0.45 0" />
         <axis
             xyz="0 0 1" />
@@ -197,6 +197,6 @@
     <!-- qianxia -->
     <xacro:thruster_macro2 thruster_id="4" parent_link="haique_link">
-        <joint_origin
-            xyz="0 0.3405 -0.0419"
+        <origin
+            xyz="0 0.3405 -0.0369"
             rpy="0.00327 0 -1.3999" />
         <axis
@@ -205,7 +205,7 @@
     <!-- zuoxia -->
     <xacro:thruster_macro1 thruster_id="5" parent_link="zuo_link">
-        <joint_origin
-            xyz="0 0.04108 0.2285"
-            rpy="1.5708 1.548 0" />
+        <origin
+            xyz="-0.005 -0.2285 0.04648 "
+            rpy="0 -0.217 0" />
         <axis
             xyz="0 0 1" />
@@ -213,6 +213,6 @@
     <!-- houxia -->
     <xacro:thruster_macro2 thruster_id="6" parent_link="haique_link">
-        <joint_origin
-            xyz="0 -0.3005 -0.0419"
+        <origin
+            xyz="0 -0.3005 -0.0369"
             rpy="0 0 0.47674" />
         <axis
@@ -221,7 +221,7 @@
     <!-- youxia -->
     <xacro:thruster_macro1 thruster_id="7" parent_link="you_link">
-        <joint_origin
-            xyz="-0.2285 -0.0379 0"
-            rpy="1.5708 -0.121 3.1416" />
+        <origin
+            xyz="-0.02387 -0.2285 0.04"
+            rpy="0 -0.45 0" />
         <axis
             xyz="0 0 -1" />

Commit message: pid adjustment complete

File: urdf/robots/haique_description/urdf/haique.xacro (robot description, xacro)
@@ -76,6 +76,18 @@
         <parent link="$(arg namespace)/haique_link" />
         <child link="$(arg namespace)/zuo_link" />
-        <axis xyz="0 1 0" />
+        <axis xyz="0 -1 0" />
+        <limit effort="4" velocity="300" />
     </joint>
+    <!-- zuoqingzhuan_joint Transmission -->
+    <transmission name="$(arg namespace)/zuoqingzhuan_tran">
+        <type>transmission_interface/SimpleTransmission</type>
+        <joint name="$(arg namespace)/zuoqingzhuan_joint">
+            <hardwareInterface>hardware_interface/EffortJointInterface</hardwareInterface>
+        </joint>
+        <actuator name="$(arg namespace)/zuoqingzhuan_motor">
+            <hardwareInterface>hardware_interface/EffortJointInterface</hardwareInterface>
+            <mechanicalReduction>1</mechanicalReduction>
+        </actuator>
+    </transmission>
     <link name="$(arg namespace)/you_link">
         <inertial>
@@ -109,11 +121,23 @@
         <parent link="$(arg namespace)/haique_link" />
         <child link="$(arg namespace)/you_link" />
+        <limit effort="4" velocity="300" />
     </joint>
+    <!-- youqingzhuan_joint Transmission -->
+    <transmission name="$(arg namespace)/youqingzhuan_tran">
+        <type>transmission_interface/SimpleTransmission</type>
+        <joint name="$(arg namespace)/youqingzhuan_joint">
+            <hardwareInterface>hardware_interface/EffortJointInterface</hardwareInterface>
+        </joint>
+        <actuator name="$(arg namespace)/youqingzhuan_motor">
+            <hardwareInterface>hardware_interface/EffortJointInterface</hardwareInterface>
+            <mechanicalReduction>1</mechanicalReduction>
+        </actuator>
+    </transmission>
      <!-- Default joint state publisher -->
     <gazebo>
-    <plugin name="uuv_joint_state_publisher" filename="libuuv_joint_state_publisher.so">
-        <robotNamespace>$(arg namespace)</robotNamespace>
-        <updateRate>50</updateRate>
-    </plugin>
+        <plugin name="uuv_joint_state_publisher" filename="libuuv_joint_state_publisher.so">
+            <robotNamespace>$(arg namespace)</robotNamespace>
+            <updateRate>50</updateRate>
+        </plugin>
     </gazebo>
     <gazebo>
